Commit message: ur10e urdf with rotated values

File: src/ur10_e_table/urdf/ur10e.urdf (robot description, URDF)
Before this commit: robot ur10e, 11 links, 10 joints
Joints:
- joint ee_fixed_joint: origin xyz=0.0 0.117 0.0 rpy=-1.5707963267 0.0 0.0 -> xyz=0.0 0.117 0.0 rpy=0.0 0.0 1.57079632679
- joint shoulder_pan_joint: origin xyz=0.0 0.0 0.181 rpy=0.0 0.0 -3.14159265359 -> xyz=0.0 0.0 0.181 rpy=0.0 0.0 0.0
