Commit message: update for abb 6700 150 320

File: src/abb_irb4600_40_255/abb_fabtory/urdf/abb_fabtory.urdf (robot description, URDF)
Before this commit: robot abb_irb6700_150_320, 12 links, 11 joints
Links:
- added link axis, mass 120; collision mesh filename=package://abb_fabtory/meshes/collision/axis_abb_irb6700.stl; visual mesh filename=package://abb_fabtory/meshes/visual/axis_abb_irb6700.stl
- added link cart, mass 120.00000; collision mesh filename=package://abb_fabtory/meshes/collision/cart_abb_irb6700.stl; visual mesh filename=package://abb_fabtory/meshes/visual/cart_abb_irb6700.stl
- added link world
- link base_link: geometry collision mesh filename=package://abb_irb6700_150_320/meshes/irb6700/collision/base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; visual mesh filename=package://abb_irb6700_150_320/meshes/irb6700/visual/base_li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
- link cylinder: geometry collision mesh filename=package://abb_irb6700_150_320/meshes/irb6700/collision/cyli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; visual mesh filename=package://abb_irb6700_150_320/meshes/irb6700/visual/cylinde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
- link link_1: geometry collision mesh filename=package://abb_irb6700_150_320/meshes/irb6700/collision/link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; visual mesh filename=package://abb_irb6700_150_320/meshes/irb6700/visual/link_1.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
- link link_2: geometry collision mesh filename=package://abb_irb6700_150_320/meshes/irb6700_150_320/collis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; visual mesh filename=package://abb_irb6700_150_320/meshes/irb6700_150_320/visual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
- link link_3: geometry collision mesh filename=package://abb_irb6700_150_320/meshes/irb6700_150_320/collis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; visual mesh filename=package://abb_irb6700_150_320/meshes/irb6700_150_320/visual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
- link link_4: geometry collision mesh filename=package://abb_irb6700_150_320/meshes/irb6700_150_320/collis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; visual mesh filename=package://abb_irb6700_150_320/meshes/irb6700_150_320/visual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
- link link_5: geometry collision mesh filename=package://abb_irb6700_150_320/meshes/irb6700/collision/link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; visual mesh filename=package://abb_irb6700_150_320/meshes/irb6700/visual/link_5.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
- link link_6: geometry collision mesh filename=package://abb_irb6700_150_320/meshes/irb6700/collision/link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; visual mesh filename=package://abb_irb6700_150_320/meshes/irb6700/visual/link_6.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
- link piston: geometry collision mesh filename=package://abb_irb6700_150_320/meshes/irb6700/collision/pist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; visual mesh filename=package://abb_irb6700_150_320/meshes/irb6700/visual/piston.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
Joints:
- added joint abb_joint: type fixed, parent cart, child base_link, origin xyz=0 0 0  rpy=0 0 0 
- added joint axis_joint: type prismatic, parent axis, child cart, origin xyz=0 0 0 rpy=0 0 0 , axis 1 0 0, limit lower=0.0 upper=4.2 effort=100000 velocity=2.618
- added joint world_joint: type fixed, parent world, child axis, origin xyz=0.0 0.0 0.0 rpy=0.0 0.0 0.0

File: src/abb_irb6700_150_320/urdf/irb6700_150_320.urdf (robot description, URDF)
Before this commit: robot abb_fabtory, 15 links, 14 joints
Links:
- removed link axis
- removed link cart
- removed link world
- link base_link: geometry collision mesh filename=package://abb_irb6700_150_320/meshes/irb6700/collision/base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; visual mesh filename=package://abb_irb6700_150_320/meshes/irb6700/visual/base_li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
- link cylinder: geometry collision mesh filename=package://abb_irb6700_150_320/meshes/irb6700/collision/cyli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; visual mesh filename=package://abb_irb6700_150_320/meshes/irb6700/visual/cylinde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
- link link_1: geometry collision mesh filename=package://abb_irb6700_150_320/meshes/irb6700/collision/link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; visual mesh filename=package://abb_irb6700_150_320/meshes/irb6700/visual/link_1.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
- link link_2: geometry collision mesh filename=package://abb_irb6700_150_320/meshes/irb6700_150_320/collis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; visual mesh filename=package://abb_irb6700_150_320/meshes/irb6700_150_320/visual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
- link link_3: geometry collision mesh filename=package://abb_irb6700_150_320/meshes/irb6700_150_320/collis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; visual mesh filename=package://abb_irb6700_150_320/meshes/irb6700_150_320/visual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
- link link_4: geometry collision mesh filename=package://abb_irb6700_150_320/meshes/irb6700_150_320/collis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; visual mesh filename=package://abb_irb6700_150_320/meshes/irb6700_150_320/visual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
- link link_5: geometry collision mesh filename=package://abb_irb6700_150_320/meshes/irb6700/collision/link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; visual mesh filename=package://abb_irb6700_150_320/meshes/irb6700/visual/link_5.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
- link link_6: geometry collision mesh filename=package://abb_irb6700_150_320/meshes/irb6700/collision/link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; visual mesh filename=package://abb_irb6700_150_320/meshes/irb6700/visual/link_6.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
- link piston: geometry collision mesh filename=package://abb_irb6700_150_320/meshes/irb6700/collision/pist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; visual mesh filename=package://abb_irb6700_150_320/meshes/irb6700/visual/piston.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
Joints:
- removed joint abb_joint
- removed joint axis_joint
- removed joint world_joint

File: src/abb_irb6700_150_320/urdf/irb6700_150_320.xacro (robot description, xacro)
@@ -1,5 +1,5 @@
 <?xml version="1.0" ?>
 <robot name="abb_irb6700_150_320" xmlns:xacro="http://ros.org/wiki/xacro">
-  <xacro:include filename="$(find abb_irb6700_support)/urdf/irb6700_150_320_macro.xacro"/>
+  <xacro:include filename="$(find abb_irb6700_150_320)/urdf/irb6700_150_320_macro.xacro"/>
   <xacro:abb_irb6700_150_320 prefix=""/>
 </robot>

File: src/abb_irb6700_150_320/urdf/irb6700_150_320_macro.xacro (robot description, xacro)
@@ -8,12 +8,12 @@
         <origin xyz="0 0 0" rpy="0 0 0" />
         <geometry>
-          <mesh filename="package://abb_irb6700_support/meshes/irb6700/visual/base_link.stl" />
-        </geometry>
-        <xacro:material_abb_white/>
-      </visual>
-      <collision>
-        <origin xyz="0 0 0" rpy="0 0 0" />
-        <geometry>
-          <mesh filename="package://abb_irb6700_support/meshes/irb6700/collision/base_link.stl" />
+          <mesh filename="package://abb_irb6700_150_320/meshes/irb6700/visual/base_link.stl" />
+        </geometry>
+        <xacro:material_abb_white/>
+      </visual>
+      <collision>
+        <origin xyz="0 0 0" rpy="0 0 0" />
+        <geometry>
+          <mesh filename="package://abb_irb6700_150_320/meshes/irb6700/collision/base_link.stl" />
         </geometry>
         <xacro:material_abb_yellow/>
@@ -24,12 +24,12 @@
         <origin xyz="0 0 0" rpy="0 0 0" />
         <geometry>
-          <mesh filename="package://abb_irb6700_support/meshes/irb6700/visual/link_1.stl" />
-        </geometry>
-        <xacro:material_abb_white/>
-      </visual>
-      <collision>
-        <origin xyz="0 0 0" rpy="0 0 0" />
-        <geometry>
-          <mesh filename="package://abb_irb6700_support/meshes/irb6700/collision/link_1.stl" />
+          <mesh filename="package://abb_irb6700_150_320/meshes/irb6700/visual/link_1.stl" />
+        </geometry>
+        <xacro:material_abb_white/>
+      </visual>
+      <collision>
+        <origin xyz="0 0 0" rpy="0 0 0" />
+        <geometry>
+          <mesh filename="package://abb_irb6700_150_320/meshes/irb6700/collision/link_1.stl" />
         </geometry>
         <xacro:material_abb_yellow/>
@@ -40,12 +40,12 @@
         <origin xyz="0 0 0" rpy="0 0 0" />
         <geometry>
-          <mesh filename="package://abb_irb6700_support/meshes/irb6700/visual/cylinder.stl" />
-        </geometry>
-        <xacro:material_abb_white/>
-      </visual>
-      <collision>
-        <origin xyz="0 0 0" rpy="0 0 0" />
-        <geometry>
-          <mesh filename="package://abb_irb6700_support/meshes/irb6700/collision/cylinder.stl" />
+          <mesh filename="package://abb_irb6700_150_320/meshes/irb6700/visual/cylinder.stl" />
+        </geometry>
+        <xacro:material_abb_white/>
+      </visual>
+      <collision>
+        <origin xyz="0 0 0" rpy="0 0 0" />
+        <geometry>
+          <mesh filename="package://abb_irb6700_150_320/meshes/irb6700/collision/cylinder.stl" />
         </geometry>
         <xacro:material_abb_yellow/>
@@ -56,12 +56,12 @@
         <origin xyz="0 0 0" rpy="0 0 0" />
         <geometry>
-          <mesh filename="package://abb_irb6700_support/meshes/irb6700/visual/piston.stl" />
-        </geometry>
-        <xacro:material_abb_white/>
-      </visual>
-      <collision>
-        <origin xyz="0 0 0" rpy="0 0 0" />
-        <geometry>
-          <mesh filename="package://abb_irb6700_support/meshes/irb6700/collision/piston.stl" />
+          <mesh filename="package://abb_irb6700_150_320/meshes/irb6700/visual/piston.stl" />
+        </geometry>
+        <xacro:material_abb_white/>
+      </visual>
+      <collision>
+        <origin xyz="0 0 0" rpy="0 0 0" />
+        <geometry>
+          <mesh filename="package://abb_irb6700_150_320/meshes/irb6700/collision/piston.stl" />
         </geometry>
         <xacro:material_abb_yellow/>
@@ -72,12 +72,12 @@
         <origin xyz="0 0 0" rpy="0 0 0" />
         <geometry>
-          <mesh filename="package://abb_irb6700_support/meshes/irb6700_150_320/visual/link_2.stl" />
-        </geometry>
-        <xacro:material_abb_white/>
-      </visual>
-      <collision>
-        <origin xyz="0 0 0" rpy="0 0 0" />
-        <geometry>
-          <mesh filename="package://abb_irb6700_support/meshes/irb6700_150_320/collision/link_2.stl" />
+          <mesh filename="package://abb_irb6700_150_320/meshes/irb6700_150_320/visual/link_2.stl" />
+        </geometry>
+        <xacro:material_abb_white/>
+      </visual>
+      <collision>
+        <origin xyz="0 0 0" rpy="0 0 0" />
+        <geometry>
+          <mesh filename="package://abb_irb6700_150_320/meshes/irb6700_150_320/collision/link_2.stl" />
         </geometry>
         <xacro:material_abb_yellow/>
@@ -88,12 +88,12 @@
         <origin xyz="0 0 0" rpy="0 0 0" />
         <geometry>
-          <mesh filename="package://abb_irb6700_support/meshes/irb6700_150_320/visual/link_3.stl" />
-        </geometry>
-        <xacro:material_abb_white/>
-      </visual>
-      <collision>
-        <origin xyz="0 0 0" rpy="0 0 0" />
-        <geometry>
-          <mesh filename="package://abb_irb6700_support/meshes/irb6700_150_320/collision/link_3.stl" />
+          <mesh filename="package://abb_irb6700_150_320/meshes/irb6700_150_320/visual/link_3.stl" />
+        </geometry>
+        <xacro:material_abb_white/>
+      </visual>
+      <collision>
+        <origin xyz="0 0 0" rpy="0 0 0" />
+        <geometry>
+          <mesh filename="package://abb_irb6700_150_320/meshes/irb6700_150_320/collision/link_3.stl" />
         </geometry>
         <xacro:material_abb_yellow/>
@@ -104,12 +104,12 @@
         <origin xyz="0 0 0" rpy="0 0 0" />
         <geometry>
-          <mesh filename="package://abb_irb6700_support/meshes/irb6700_150_320/visual/link_4.stl" />
-        </geometry>
-        <xacro:material_abb_white/>
-      </visual>
-      <collision>
-        <origin xyz="0 0 0" rpy="0 0 0" />
-        <geometry>
-          <mesh filename="package://abb_irb6700_support/meshes/irb6700_150_320/collision/link_4.stl" />
+          <mesh filename="package://abb_irb6700_150_320/meshes/irb6700_150_320/visual/link_4.stl" />
+        </geometry>
+        <xacro:material_abb_white/>
+      </visual>
+      <collision>
+        <origin xyz="0 0 0" rpy="0 0 0" />
+        <geometry>
+          <mesh filename="package://abb_irb6700_150_320/meshes/irb6700_150_320/collision/link_4.stl" />
         </geometry>
         <xacro:material_abb_yellow/>
@@ -120,12 +120,12 @@
         <origin xyz="0 0 0" rpy="0 0 0" />
         <geometry>
-          <mesh filename="package://abb_irb6700_support/meshes/irb6700/visual/link_5.stl" />
-        </geometry>
-        <xacro:material_abb_white/>
-      </visual>
-      <collision>
-        <origin xyz="0 0 0" rpy="0 0 0" />
-        <geometry>
-          <mesh filename="package://abb_irb6700_support/meshes/irb6700/collision/link_5.stl" />
+          <mesh filename="package://abb_irb6700_150_320/meshes/irb6700/visual/link_5.stl" />
+        </geometry>
+        <xacro:material_abb_white/>
+      </visual>
+      <collision>
+        <origin xyz="0 0 0" rpy="0 0 0" />
+        <geometry>
+          <mesh filename="package://abb_irb6700_150_320/meshes/irb6700/collision/link_5.stl" />
         </geometry>
         <xacro:material_abb_yellow/>
@@ -136,12 +136,12 @@
         <origin xyz="0 0 0" rpy="0 0 0" />
         <geometry>
-          <mesh filename="package://abb_irb6700_support/meshes/irb6700/visual/link_6.stl" />
-        </geometry>
-        <xacro:material_abb_white/>
-      </visual>
-      <collision>
-        <origin xyz="0 0 0" rpy="0 0 0" />
-        <geometry>
-          <mesh filename="package://abb_irb6700_support/meshes/irb6700/collision/link_6.stl" />
+          <mesh filename="package://abb_irb6700_150_320/meshes/irb6700/visual/link_6.stl" />
+        </geometry>
+        <xacro:material_abb_white/>
+      </visual>
+      <collision>
+        <origin xyz="0 0 0" rpy="0 0 0" />
+        <geometry>
+          <mesh filename="package://abb_irb6700_150_320/meshes/irb6700/collision/link_6.stl" />
         </geometry>
         <xacro:material_abb_yellow/>
